File: pcb/D4v2Charger.kicad_pcb (KiCad board)
At the start: 2 copper layers, 17 x 14 mm, 13 parts, among them J1 Conn_01x02_Pin, U1 BQ25185DLHR

Commit message: updates & license addition
Parts:
- added D3: D_Schottky, PMEG1020EJ_115:DIO_PMEG6010CEJF, F.Cu at (138.5, 96.0)
- added F1: Polyfuse, Littlefuse_0406L:0402L100SLKR, F.Cu at (138.5, 97.5)
- moved D2 1.62 mm to (148.5, 93.0), turned to 180 degrees
- moved D1 1.58 mm to (138.5, 93.0)
- moved R4 1.58 mm to (149.0, 94.5)
- moved R3 1.46 mm to (138.0, 94.5)
- moved C3 1.00 mm to (140.0, 87.5)
- moved C2 0.71 mm to (140.0, 88.5)
- moved R5 0.71 mm to (140.0, 89.5)
- moved C1 0.50 mm to (147.0, 87.0)
- moved R6 0.50 mm to (147.0, 89.0)
- moved R7 0.50 mm to (147.0, 88.0)
- moved R8 0.50 mm to (147.0, 90.0)
- moved U1 0.50 mm to (143.5, 87.5)
Connections:
- J1 pad 1: VBUS -> Net-(J1-Pin_1)
Routing:
- net GND: track 5.01 -> 0.80 mm, vias 1 -> 0
- net Net-(J1-Pin_1): track 0.00 -> 3.45 mm
- net VBUS: track 34.9 -> 37.9 mm, vias 3 -> 1
- net Net-(D2-K): track 1.83 -> 0.00 mm
- net Net-(D3-A): track 0.00 -> 1.76 mm
- net Net-(D2-A): track 11.9 -> 11.0 mm
- net Net-(D1-A): track 11.2 -> 12.0 mm

Commit message: updated pcb clearance for magnetic charger
Parts:
- moved J1 0.50 mm to (142.2, 97.5)
Changed lines of the file:
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@@
 	(footprint "Connector_PinHeader_2.54mm:PinHeader_1x02_P2.54mm_Vertical"
 		(layer "F.Cu")
-		(at 142.225001 97 90)
+		(at 142.225 97.5 90)
 		(descr "Through hole straight pin header, 1x02, 2.54mm pitch, single row")
 		(tags "Through hole pin header THT 1x02 2.54mm single row")
@@
 		(min_thickness 0.25)
 		(filled_areas_thickness no)
-		(fill
+		(fill yes
 			(thermal_gap 0.5)
 			(thermal_bridge_width 0.5)
